File: 2026_InClass_Balancing_Robot.kicad_pcb (KiCad board)
At the start: 2 copper layers, 31 parts, among them J4 CONN_MPU6050, J5 MT6701_CONN, J6 ENCODER_CONN, J7 Conn_01x04, J8 USB_C_Receptacle, SW1 SW_uP_Reset, U1 STM32F401RBTx, U2 LD1117S50TR_SOT223, U3 LD1117S50TR_SOT223, U4 TB6612FNG, U6 USBLC6-2SC6

Commit message: all files in project
layout from class
Parts:
- moved J5 103.6 mm to (249.5, 104.5), turned to -90 degrees
- moved J4 101.5 mm to (232.3, 78.0), turned to 90 degrees
- moved J6 91.6 mm to (242.0, 122.5)
- moved J7 88.0 mm to (249.0, 89.0), turned to -90 degrees
- moved C14 83.8 mm to (224.1, 94.0)
- moved C15 79.7 mm to (223.0, 88.0)
- moved C13 72.9 mm to (212.5, 73.4)
- moved C7 66.5 mm to (202.0, 92.5)
- moved U6 65.2 mm to (201.1, 117.0)
- moved C6 64.0 mm to (198.5, 97.5)
- moved C8 60.2 mm to (198.5, 86.0)
- moved C5 59.8 mm to (193.5, 97.5)
- moved C11 58.5 mm to (199.0, 81.0)
- moved C10 57.4 mm to (197.5, 69.0)
- moved U4 55.1 mm to (217.0, 122.0), turned to 90 degrees
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